File: Kicad-NANO/template.kicad_pcb (KiCad board)
At the start: 2 copper layers, 21 parts, among them J1 sensor 1, J2 sensor 2, J3 sensor 3, J4 SERVO, J5 MOTOR, J6 POWER, J7 START, P1 Digital, P2 Analog, P3 CONN_01X01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

Commit message: Ny h-brygga
Other:
- net class Default removed
