File: H-Brygga v2/H-Brygga v2.kicad_pcb (KiCad board)
At the start: 2 copper layers, 19 parts, among them J1 POWER, J2 sensor 2, J3 SERVO, J4 sensor 1, J5 START, J6 sensor 3, J7 MOTOR, P1 Digital, P2 Analog, P7 Digital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

Commit message: H-brygga
Parts:
- added C3: 0.1uF, Capacitor_THT:CP_Radial_D6.3mm_P2.50mm, F.Cu at (187.3, 93.4)
- added D5: 1N4007, Diode_THT:D_DO-41_SOD81_P10.16mm_Horizontal, F.Cu at (154.9, 85.2)
- added J8: MOTOR, Connector_Wago:Wago_734-132_1x02_P3.50mm_Vertical, F.Cu at (168.9, 93.2)
- added Q1: BC547, Package_TO_SOT_THT:TO-92_Inline, F.Cu at (191.1, 89.5)
- added R2: 150, Resistor_THT:R_Axial_DIN0207_L6.3mm_D2.5mm_P10.16mm_Horizontal, F.Cu at (186.7, 79.4)
- added R3: 10k, Resistor_THT:R_Axial_DIN0207_L6.3mm_D2.5mm_P10.16mm_Horizontal, F.Cu at (153.0, 64.2)
- added SW1: SW_MEC_5E, Rasberry 2040:SW_B3F-1000[1], F.Cu at (175.9, 73.0)
- C1: value 100uf -> C
- C2: value 0.1uF -> 100uf
- D3: value 1N4007 -> LED; footprint Diode_THT:D_DO-41_SOD81_P10.16mm_Horizontal -> LED_THT:LED_D5.0mm
- J1: value POWER -> Högtalare
- J2: value sensor 2 -> POWER; footprint Connector_JST:JST_XH_B3B-XH-A_1x03_P2.50mm_Vertical -> Connector_Wago:Wago_734-132_1x02_P3.50mm_Vertical
- J3: value SERVO -> sensor 1
- J4: value sensor 1 -> SERVO
- J5: value START -> sensor 2
- J6: value sensor 3 -> START
- J7: value MOTOR -> sensor 3; footprint Connector_Wago:Wago_734-132_1x02_P3.50mm_Vertical -> Connector_JST:JST_XH_B3B-XH-A_1x03_P2.50mm_Vertical
- P1, P2, P7, P8: footprint footprints:Socket_Strip_Arduino_1x15 -> Socket_Arduino_Nano:Socket_Strip_Arduino_1x15
- moved R1 108.4 mm to (181.6, 66.0)
- moved J6 106.2 mm to (173.9, 54.6), turned to -90 degrees
- moved J5 100.9 mm to (201.8, 54.6), turned to -90 degrees
- moved J4 98.7 mm to (180.9, 54.6), turned to -90 degrees
- moved P7 98.6 mm to (128.3, 75.7)
- moved P2 92.8 mm to (128.3, 96.0)
- moved D3 88.4 mm to (181.0, 88.3), turned to 90 degrees
- moved J3 80.8 mm to (194.9, 54.6), turned to -90 degrees
- moved J1 78.1 mm to (198.8, 93.3)
- moved U1 77.4 mm to (195.1, 66.0), turned to -90 degrees
- moved P1 70.3 mm to (128.3, 80.7)
- moved P8 63.5 mm to (128.3, 60.4)
- moved D2 62.0 mm to (154.9, 90.9), turned to 180 degrees
- moved C1 56.3 mm to (186.7, 73.6), turned to 90 degrees
- moved J2 55.6 mm to (132.7, 52.8), turned to 180 degrees
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Connections:
- net /2 renamed 2.
- net /3(**) renamed 3(**).
- net /4 renamed 4
- C1 pad 1: Vin -> 8
- C1 pad 2: GND -> Net-(C1-Pad2)
- D3 pad 1: Vin -> Net-(D3-Pad1)
- D3 pad 2: Net-(D3-Pad2) -> 7
- D4 pad 1: Net-(D3-Pad2) -> Vin
- D4 pad 2: GND -> Net-(D4-Pad2)
- J1 pad 1: GND -> +5V
- J1 pad 2: Vin -> Net-(J1-Pad2)
- J2 pad 1: +5V -> GND
- J2 pad 2: A1 -> Vin
- J3 pad 2: 6(**) -> A0
- J4 pad 2: A0 -> 6(**)
- J5 pad 2: 9(**) -> A1
- J6 pad 2: A2 -> 9(**)
- J7 pad 1: Net-(D1-Pad2) -> +5V
- J7 pad 2: Net-(D3-Pad2) -> A2
- P1 pad 1: /1(Tx) -> /1(Tx).
- P1 pad 10: 7 -> /7.
- P1 pad 11: 8 -> /8.
- P1 pad 12: 9(**) -> /9(**).
- P1 pad 13: /10(**/SS) -> /10(**/SS).
- P1 pad 14: /11(**/MOSI) -> 11(**/MOSI).
- P1 pad 15: /12(MISO) -> /12(MISO).
- P1 pad 2: /0(Rx) -> /0(Rx).
- P1 pad 3: /Reset -> /Reset.
- P1 pad 8: 5(**) -> /5(**).
- P1 pad 9: 6(**) -> /6(**).
- P2 pad 10: A2 -> /A2.
- P2 pad 11: A1 -> /A1.
- P2 pad 12: A0 -> /A0.
- P2 pad 13: /AREF -> /AREF.
- P2 pad 15: /13(SCK) -> /13(SCK).
- P2 pad 3: /Reset -> /Reset.
- P2 pad 5: /A7 -> /A7.
- P2 pad 6: /A6 -> /A6.
- P2 pad 7: /A5 -> /A5.
- P2 pad 8: /A4 -> /A4.
- P2 pad 9: /A3 -> /A3.
- U1 pad 3: Net-(D3-Pad2) -> Net-(D4-Pad2)
- U1 pad 9: unconnected-(U1-Pad9) -> +5V
Routing:
- net (no net): track 0.00 -> 217.9 mm

Commit message: H-brygga
Parts:
- moved R3 116.4 mm to (252.0, 125.6), turned to 90 degrees
- moved R1 69.3 mm to (156.0, 130.4), turned to -90 degrees
- moved J5 55.7 mm to (147.7, 41.5), turned to 90 degrees
- moved D3 55.3 mm to (177.5, 143.5)
- moved C3 52.3 mm to (215.0, 137.8)
- moved J7 49.3 mm to (140.5, 41.5), turned to 90 degrees
- moved J3 42.3 mm to (154.7, 41.5), turned to 90 degrees
- moved C2 39.3 mm to (198.5, 128.3)
- moved J8 32.8 mm to (200.7, 84.9), turned to 90 degrees
- moved R2 30.1 mm to (187.5, 109.4)
- moved J4 17.9 mm to (168.7, 41.5), turned to 90 degrees
- moved J6 17.9 mm to (161.8, 41.5), turned to 90 degrees
- moved C1 16.3 mm to (172.1, 80.8), turned to 0 degrees
- moved D5 12.4 mm to (142.5, 85.2), turned to 0 degrees
- moved U1 10.7 mm to (195.7, 55.4)
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Connections:
- net 3(**). renamed 3(**)
- net 4 renamed 4.
- C1 pad 1: 8 -> 7a
- D3 pad 2: 7 -> 8a
- J3 pad 1: +5V -> A0
- J3 pad 2: A0 -> +5V
- J4 pad 1: +5V -> 6(**)
- J4 pad 2: 6(**) -> +5V
- J5 pad 1: +5V -> A1
- J5 pad 2: A1 -> +5V
- J6 pad 1: +5V -> 5(**)
- J6 pad 2: 9(**) -> +5V
- J7 pad 1: +5V -> A2
- J7 pad 2: A2 -> +5V
- P7 pad 10: 7 -> 7a
- P7 pad 11: 8 -> 8a
- R1 pad 1: 9(**) -> 5(**)
- R3 pad 2: 8 -> 7a
- SW1 pad 3: 8 -> 7a
- U1 pad 5: 8 -> 8a
- U1 pad 6: 5(**) -> 9(**)
- U1 pad 7: 7 -> 7a
Routing:
- net GND: track 0.00 -> 118.6 mm
- net +5V: track 0.00 -> 61.9 mm
- net 7a: track 0.00 -> 59.5 mm
- net Vin: track 0.00 -> 51.1 mm
- net 9(**): track 0.00 -> 48.7 mm
- net 8a: track 0.00 -> 47.1 mm
- net 5(**): track 0.00 -> 45.3 mm
- net 6(**): track 0.00 -> 42.5 mm
- net (no net): track 217.9 -> 191.3 mm
- net A2: track 0.00 -> 19.4 mm
- net A1: track 0.00 -> 17.5 mm
- net A0: track 0.00 -> 15.6 mm
- net Net-(C1-Pad2): track 0.00 -> 10.7 mm
- net 4.: track 0.00 -> 9.01 mm
- net 3(**): track 0.00 -> 9.01 mm
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
Commit message: Brygga
Parts:
- added REF**: MountingHole_3mm, MountingHole:MountingHole_3mm, F.Cu at (187.5, 51.1)
- added REF**: MountingHole_3mm, MountingHole:MountingHole_3mm, F.Cu at (169.6, 93.7)
- moved D3 86.3 mm to (179.5, 57.2), turned to 0 degrees
- moved R3 81.5 mm to (188.6, 74.3)
- moved J2 71.6 mm to (202.4, 48.7), turned to 90 degrees
- moved R1 66.4 mm to (146.1, 64.8), turned to 180 degrees
- moved R2 61.9 mm to (175.0, 48.8)
- moved C3 55.5 mm to (201.9, 83.9)
- moved D1 53.0 mm to (180.7, 100.1), turned to 90 degrees
- moved C2 51.5 mm to (201.9, 76.9)
- moved D4 48.9 mm to (175.6, 100.1), turned to 90 degrees
- moved D2 39.3 mm to (192.2, 86.6), turned to 90 degrees
- moved D5 30.2 mm to (172.7, 84.1)
- moved Q1 14.7 mm to (173.4, 78.7)
- moved C1 13.2 mm to (169.0, 67.9)
- moved J1 11.0 mm to (191.1, 93.4)
- moved J5 9.31 mm to (147.3, 50.8)
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Routing:
- net Vin: track 51.1 -> 247.8 mm
- net (no net): track 191.3 -> 0.00 mm
- net GND: track 118.6 -> 268.6 mm
- net +5V: track 61.9 -> 183.4 mm
- net Net-(D4-Pad2): track 0.00 -> 94.0 mm
- net Net-(D1-Pad2): track 0.00 -> 65.8 mm
- net Net-(J1-Pad2): track 0.00 -> 31.1 mm
- net 11(**/MOSI).: track 0.00 -> 13.4 mm
- net 6(**): track 42.5 -> 33.3 mm
- net A0: track 15.6 -> 6.46 mm
- net A1: track 17.5 -> 8.75 mm
- net 7a: track 59.5 -> 53.3 mm
- net A2: track 19.4 -> 13.4 mm
- net Net-(D3-Pad1): track 0.00 -> 5.26 mm
- net 8a: track 47.1 -> 50.4 mm
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Other:
- board outline added: 83.8 x 66.2 mm

Commit message: h-brygga
Parts:
- moved REF** 23.3 mm to (146.9, 88.5)
- moved REF** 2.51 mm to (189.8, 50.1)
- moved Q1 1.94 mm to (173.0, 76.8), turned to -90 degrees
- moved R3 0.72 mm to (188.5, 73.6)
Connections:
- P1 pad 13: /10(**/SS). -> 10(**/SS).
- P1 pad 15: /12(MISO). -> 12(MISO).
- P7 pad 13: /10(**/SS) -> 10(**/SS).
- P7 pad 15: /12(MISO) -> 12(MISO).
Routing:
- net 12(MISO).: track 0.00 -> 9.01 mm
- net 10(**/SS).: track 0.00 -> 9.01 mm
- net GND: track 268.6 -> 276.6 mm
- net Net-(J1-Pad2): track 31.1 -> 38.8 mm
- net 11(**/MOSI).: track 13.4 -> 18.5 mm
- net 7a: track 53.3 -> 52.2 mm
- net +5V: track 183.4 -> 182.7 mm
Other:
- board size 83.8 x 66.2 mm -> 83.8 x 64.2 mm
