File: H-Brygga v2/H-Brygga v2.kicad_sch (KiCad schematic)
At the start: 27 parts, among them J1 POWER, J2 sensor 2, J3 SERVO, J4 sensor 1, J5 START, J6 sensor 3, J7 MOTOR, P10 CONN_01X01, P11 CONN_01X01, P12 CONN_01X01, P3 CONN_01X01, P4 CONN_01X01, P5 CONN_01X01, P6 CONN_01X01, P9 CONN_01X01, U1 L298HN

Commit message: H-brygga
Parts:
- added C1: (no value), symbol Device:C
- added D3: (no value), symbol Device:LED
- added J1: (no value), symbol Connector:Conn_01x02_Female
- added Q1: (no value), symbol Transistor_BJT:BC547
- added R2, R3: (no value), symbol Device:R
- added SW1: (no value), symbol Switch:SW_MEC_5E
- renumbered C1 to C2, C2 to C3, D3 to D4, D4 to D5, J1 to J2, J4 to J3, J3 to J4, J2 to J5, J5 to J6, J6 to J7, J7 to J8
Connections:
- net +5V: now also U1.9 (Vss), J1.1 (Pin_1), SW1.1
- net 0(Rx): no longer P1.2 (Pin_2)
- net 1(Tx): no longer P1.1 (Pin_1)
- net 10(**/SS): no longer P1.13 (Pin_13)
- net 11(**/MOSI): no longer P1.14 (Pin_14)
- net 12(MISO): no longer P1.15 (Pin_15)
- net 13(SCK): no longer P2.15 (Pin_15)
- net 5(**): no longer P1.8 (Pin_8)
- net 6(**): no longer P1.9 (Pin_9)
- net 7: now also D3.2 (A); no longer P1.10 (Pin_10)
- net 8: now also C1.1, R3.2, SW1.3 (K); no longer P1.11 (Pin_11)
- net 9(**): no longer P1.12 (Pin_12)
- net A0: no longer P2.12 (Pin_12)
- net A1: no longer P2.11 (Pin_11)
- net A2: no longer P2.10 (Pin_10)
- net A3: no longer P2.9 (Pin_9)
- net A4: no longer P2.8 (Pin_8)
- net A5: no longer P2.7 (Pin_7)
- net A6: no longer P2.6 (Pin_6)
- net A7: no longer P2.5 (Pin_5)
- net AREF: no longer P2.13 (Pin_13)
- net GND: now also Q1.3 (E), R2.1, R3.1
- net Reset: no longer P1.3 (Pin_3), P2.3 (Pin_3)
- new net: J1.2 (Pin_2), Q1.1 (C)
- new net: C1.2, SW1.2
- new net: D3.1 (K), R2.2
- new net 0(Rx).: P1.2 (Pin_2)
- new net 1(Tx).: P1.1 (Pin_1)
- new net 10(**/SS).: P1.13 (Pin_13)
- new net 11(**/MOSI).: P1.14 (Pin_14), Q1.2 (B)
- new net 12(MISO).: P1.15 (Pin_15)
- new net 13(SCK).: P2.15 (Pin_15)
- new net 5(**).: P1.8 (Pin_8)
- new net 6(**).: P1.9 (Pin_9)
- new net 7.: P1.10 (Pin_10)
- new net 8.: P1.11 (Pin_11)
- new net 9(**).: P1.12 (Pin_12)
- new net A0.: P2.12 (Pin_12)
- new net A1.: P2.11 (Pin_11)
- new net A2.: P2.10 (Pin_10)
- new net A3.: P2.9 (Pin_9)
- new net A4.: P2.8 (Pin_8)
- new net A5.: P2.7 (Pin_7)
- new net A6.: P2.6 (Pin_6)
- new net A7.: P2.5 (Pin_5)
- new net AREF.: P2.13 (Pin_13)
- new net Reset.: P1.3 (Pin_3), P2.3 (Pin_3)
Other:
- moved on the sheet: J3, J5

Commit message: H-brygga
Parts:
- C1: value (none) -> C; footprint (none) -> Capacitor_THT:CP_Radial_D6.3mm_P2.50mm
- D3: value (none) -> LED; footprint (none) -> LED_THT:LED_D5.0mm
- J1: value (none) -> Högtalare; footprint (none) -> Connector_Wago:Wago_734-132_1x02_P3.50mm_Vertical
- P1, P7: value (none) -> Digital; footprint (none) -> Socket_Arduino_Nano:Socket_Strip_Arduino_1x15
- P2, P8: value (none) -> Analog; footprint (none) -> Socket_Arduino_Nano:Socket_Strip_Arduino_1x15
- Q1: value (none) -> BC547; footprint (none) -> Package_TO_SOT_THT:TO-92_Inline
- R2: value (none) -> 150; footprint (none) -> Resistor_THT:R_Axial_DIN0207_L6.3mm_D2.5mm_P10.16mm_Horizontal
- R3: value (none) -> 10k; footprint (none) -> Resistor_THT:R_Axial_DIN0207_L6.3mm_D2.5mm_P10.16mm_Horizontal
- SW1: value (none) -> SW_MEC_5E; footprint (none) -> Rasberry 2040:SW_B3F-1000[1]
Connections:
- net +5V: now also J3.2 (Pin_2), J4.2 (Pin_2), J5.2 (Pin_2), J6.2 (Pin_2), J7.2 (Pin_2); no longer J3.1 (Pin_1), J4.1 (Pin_1), J5.1 (Pin_1), J6.1 (Pin_1), J7.1 (Pin_1)
- net 5(**): now also J6.1 (Pin_1), R1.1; no longer U1.6 (EnA)
- net 6(**): now also J4.1 (Pin_1); no longer J4.2 (Pin_2)
- net 9(**): now also U1.6 (EnA); no longer J6.2 (Pin_2), R1.1
- net A0: now also J3.1 (Pin_1); no longer J3.2 (Pin_2)
- net A1: now also J5.1 (Pin_1); no longer J5.2 (Pin_2)
- net A2: now also J7.1 (Pin_1); no longer J7.2 (Pin_2)
- net 2 renamed 2.
- net 4 renamed 4.
- net 7 renamed 7a
- net 7a: now also C1.1, R3.2, SW1.3 (K); no longer D3.2 (A)
- removed net 8: C1.1, P7.11 (Pin_11), R3.2, SW1.3 (K), U1.5 (IN1)
- new net 8a: D3.2 (A), P7.11 (Pin_11), U1.5 (IN1)
Other:
- moved on the sheet: C1, D3, J1, J3, Q1, R1, R2, R3, SW1

Commit message: h-brygga
Connections:
- net 12(MISO). is gone; now on net 12(MISO): P1.15 (Pin_15)
- net 10(**/SS). renamed 10(**/SS)
Changed lines of the file:
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@@
+    )
+  )
+  (global_label "12(MISO)" (shape input) (at 106.68 50.8 180) (fields_autoplaced)
+    (effects (font (size 1.27 1.27)) (justify right))
+    (property "Intersheet References" "${INTERSHEET_REFS}" (id 0) (at 95.5583 50.8794 0)
+      (effects (font (size 1.27 1.27)) (justify right) hide)
     )
   )
@@
     )
   )
+  (global_label "10(**{slash}SS)." (shape input) (at 106.68 46.99 0) (fields_autoplaced)
+    (effects (font (size 1.27 1.27)) (justify left))
+    (property "Intersheet References" "${INTERSHEET_REFS}" (id 0) (at 119.495 46.9106 0)
+      (effects (font (size 1.27 1.27)) (justify left) hide)
+    )
+  )
+  (global_label "12(MISO)." (shape input) (at 106.68 50.8 0) (fields_autoplaced)
+    (effects (font (size 1.27 1.27)) (justify left))
+    (property "Intersheet References" "${INTERSHEET_REFS}" (id 0) (at 118.4064 50.7206 0)
+      (effects (font (size 1.27 1.27)) (justify left) hide)
+    )
+  )
   (global_label "3(**)" (shape input) (at 106.68 39.37 180) (fields_autoplaced)
     (effects (font (size 1.27 1.27)) (justify right))
@@
     (property "Intersheet References" "${INTERSHEET_REFS}" (id 0) (at 2.54 0 0)
       (effects (font (size 1.27 1.27)) hide)
+    )
+  )
+  (global_label "10(**{slash}SS)" (shape input) (at 106.68 46.99 180) (fields_autoplaced)
+    (effects (font (size 1.27 1.27)) (justify right))
+    (property "Intersheet References" "${INTERSHEET_REFS}" (id 0) (at 94.4698 46.9106 0)
+      (effects (font (size 1.27 1.27)) (justify right) hide)
     )
   )
@@
       (effects (font (size 1.27 1.27)) hide)
     )
-    (property "Value" "" (id 1) (at 246.38 124.4599 90)
+    (property "Value" "GND" (id 1) (at 246.38 124.4599 90)
       (effects (font (size 1.27 1.27)) (justify right))
     )

Commit message: h-brygga
Parts:
- Q1: value BC547 -> (none); footprint Package_TO_SOT_THT:TO-92_Inline -> (none)
Changed lines of the file:
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@@
       (effects (font (size 1.27 1.27)) (justify left))
     )
-    (property "Value" "BC547" (id 1) (at 205.74 148.5901 0)
+    (property "Value" "" (id 1) (at 205.74 148.5901 0)
       (effects (font (size 1.27 1.27)) (justify left))
     )
-    (property "Footprint" "Package_TO_SOT_THT:TO-92_Inline" (id 2) (at 205.74 147.955 0)
+    (property "Footprint" "" (id 2) (at 205.74 147.955 0)
       (effects (font (size 1.27 1.27) italic) (justify left) hide)
     )
