File: H-Brygga v3/H-brygga V3/H-brygga V3.kicad_pcb (KiCad board)
At the start: 2 copper layers, 78.2 x 63.2 mm, 31 parts, among them J1 POWER, J2 sensor vänster, J3 SERVO, J4 sensor motor, J5 START, J6 sensor höger, J7 MOTOR, P1 Digital, P2 Analog, P7 Digital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

Commit message: H-brygga v3
Parts:
- added J8: Högtalare, Connector_Wago:Wago_734-132_1x02_P3.50mm_Vertical, F.Cu at (99.7, 104.1)
- added U2: DFR0299, footprints:DIPS1778W50P254L2100H170Q16N, F.Cu at (98.3, 79.3)
Changed lines of the file:
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@@
   (net 64 "11(**{slash}MOSI)")
   (net 65 "/7a")
+  (net 66 "Net-(J8-Pad1)")
+  (net 67 "Net-(J8-Pad2)")
+  (net 68 "MP3+")
+  (net 69 "unconnected-(U2-Pad2)")
+  (net 70 "unconnected-(U2-Pad3)")
+  (net 71 "unconnected-(U2-Pad4)")
+  (net 72 "unconnected-(U2-Pad5)")
+  (net 73 "Previous")
+  (net 74 "Next")
+  (net 75 "unconnected-(U2-Pad12)")
+  (net 76 "unconnected-(U2-Pad13)")
+  (net 77 "unconnected-(U2-Pad14)")
+  (net 78 "unconnected-(U2-Pad15)")
+  (net 79 "unconnected-(U2-Pad16)")
   (footprint "Connector_JST:JST_XH_B3B-XH-A_1x03_P2.50mm_Vertical" (layer "F.Cu")
     (at 62.4 87.5 90)
@@
     )
   )
+  (footprint "footprints:DIPS1778W50P254L2100H170Q16N" (layer "F.Cu")
+    (at 98.31 79.31)
+    (descr "MP3-TF-16P")
+    (tags "Undefined or Miscellaneous")
+    (property "Arrow Part Number" "DFR0299")
+    (property "Arrow Price/Stock" "https://www.arrow.com/en/products/dfr0299/dfrobot?region=nac")
+    (property "Description" "DFRobot Accessories DFPlayer")
+    (property "Height" "1.7")
+    (property "Manufacturer_Name" "DFRobot")
+    (property "Manufacturer_Part_Number" "DFR0299")
+    (property "Mouser Part Number" "426-DFR0299")
+    (property "Mouser Price/Stock" "https://www.mouser.co.uk/ProductDetail/DFRobot/DFR0299?qs=Zcin8yvlhnPSNhqM2hweWw%3D%3D")
+    (property "Sheetfile" "H-brygga V3.kicad_sch")
+    (property "Sheetname" "")
+    (attr through_hole)
+    (fp_text reference "U2" (at 0 0) (layer "F.SilkS")
+      (effects (font (size 1.27 1.27) (thickness 0.254)))
+    )
+    (fp_text value "DFR0299" (at 0 0) (layer "F.SilkS") hide
+      (effects (font (size 1.27 1.27) (thickness 0.254)))
+    )
+    (fp_text user "${REFERENCE}" (at 0 0) (layer "F.Fab")
+      (effects (font (size 1.27 1.27) (thickness 0.254)))
+    )
+    (fp_line (start -1.61 19.39) (end 19.39 19.39) (layer "F.SilkS") (width 0.2))
+    (fp_line (start 19.39 -1.61) (end -1.61 -1.61) (layer "F.SilkS") (width 0.2))
+    (fp_line (start -1.61 -1.61) (end -1.61 0) (layer "F.SilkS") (width 0.2))
+    (fp_line (start 19.64 -1.86) (end 19.64 19.64) (layer "F.CrtYd") (width 0.05))
+    (fp_line (start -1.86 19.64) (end -1.86 -1.86) (layer "F.CrtYd") (width 0.05))
+    (fp_line (start -1.86 -1.86) (end 19.64 -1.86) (layer "F.CrtYd") (width 0.05))
+    (fp_line (start 19.64 19.64) (end -1.86 19.64) (layer "F.CrtYd") (width 0.05))
+    (fp_line (start 19.39 -1.61) (end 19.39 19.39) (layer "F.Fab") (width 0.1))
+    (fp_line (start 19.39 19.39) (end -1.61 19.39) (layer "F.Fab") (width 0.1))
+    (fp_line (start -1.61 -1.61) (end 19.39 -1.61) (layer "F.Fab") (width 0.1))
+    (fp_line (start -1.61 19.39) (end -1.61 -1.61) (layer "F.Fab") (width 0.1))
+    (fp_line (start -1.61 -0.34) (end -0.34 -1.61) (layer "F.Fab") (width 0.1))
+    (pad "1" thru_hole rect (at 0 0) (size 1.35 1.35) (drill 0.9) (layers *.Cu *.Mask)
+      (net 68 "MP3+") (pinfunction "VCC") (pintype "power_in"))
+    (pad "2" thru_hole circle (at 0 2.54) (size 1.35 1.35) (drill 0.9) (layers *.Cu *.Mask)
+      (net 69 "unconnected-(U2-Pad2)") (pinfunction "RX") (pintype "input"))
+    (pad "3" thru_hole circle (at 0 5.08) (size 1.35 1.35) (drill 0.9) (layers *.Cu *.Mask)
+      (net 70 "unconnected-(U2-Pad3)") (pinfunction "TX") (pintype "output"))
+    (pad "4" thru_hole circle (at 0 7.62) (size 1.35 1.35) (drill 0.9) (layers *.Cu *.Mask)
+      (net 71 "unconnected-(U2-Pad4)") (pinfunction "DAC_R") (pintype "output"))
+    (pad "5" thru_hole circle (at 0 10.16) (size 1.35 1.35) (drill 0.9) (layers *.Cu *.Mask)
+      (net 72 "unconnected-(U2-Pad5)") (pinfunction "DAC_L") (pintype "output"))
+    (pad "6" thru_hole circle (at 0 12.7) (size 1.35 1.35) (drill 0.9) (layers *.Cu *.Mask)
+      (net 67 "Net-(J8-Pad2)") (pinfunction "SPK_1") (pintype "output"))
+    (pad "7" thru_hole circle (at 0 15.24) (size 1.35 1.35) (drill 0.9) (layers *.Cu *.Mask)
+      (net 2 "GND") (pinfunction "GND_1") (pintype "power_in"))
+    (pad "8" thru_hole circle (at 0 17.78) (size 1.35 1.35) (drill 0.9) (layers *.Cu *.Mask)
+      (net 66 "Net-(J8-Pad1)") (pinfunction "SPK_2") (pintype "output"))
+    (pad "9" thru_hole circle (at 17.78 17.78) (size 1.35 1.35) (drill 0.9) (layers *.Cu *.Mask)
+      (net 73 "Previous") (pinfunction "IO_1") (pintype "input"))
+    (pad "10" thru_hole circle (at 17.78 15.24) (size 1.35 1.35) (drill 0.9) (layers *.Cu *.Mask)
+      (net 2 "GND") (pinfunction "GND_2") (pintype "power_in"))
+    (pad "11" thru_hole circle (at 17.78 12.7) (size 1.35 1.35) (drill 0.9) (layers *.Cu *.Mask)
+      (net 74 "Next") (pinfunction "IO_2") (pintype "input"))
+    (pad "12" thru_hole circle (at 17.78 10.16) (size 1.35 1.35) (drill 0.9) (layers *.Cu *.Mask)
+      (net 75 "unconnected-(U2-Pad12)") (pinfunction "ADKEY_1") (pintype "input"))
+    (pad "13" thru_hole circle (at 17.78 7.62) (size 1.35 1.35) (drill 0.9) (layers *.Cu *.Mask)
+      (net 76 "unconnected-(U2-Pad13)") (pinfunction "ADKEY_2") (pintype "input"))
+    (pad "14" thru_hole circle (at 17.78 5.08) (size 1.35 1.35) (drill 0.9) (layers *.Cu *.Mask)
+      (net 77 "unconnected-(U2-Pad14)") (pinfunction "USB+") (pintype "bidirectional"))
+    (pad "15" thru_hole circle (at 17.78 2.54) (size 1.35 1.35) (drill 0.9) (layers *.Cu *.Mask)
+      (net 78 "unconnected-(U2-Pad15)") (pinfunction "USB-") (pintype "bidirectional"))
+    (pad "16" thru_hole circle (at 17.78 0) (size 1.35 1.35) (drill 0.9) (layers *.Cu *.Mask)
+      (net 79 "unconnected-(U2-Pad16)") (pinfunction "BUSY") (pintype "output"))
+  )
   (footprint "footprints:CP_Radial_D6.3mm_P2.50mm" (layer "F.Cu")
     (at 84.18238 130.4 180)
@@
       (offset (xyz 0 0 0))
       (scale (xyz 1 1 1))
+      (rotate (xyz 0 0 0))
+    )
+  )
+  (footprint "Connector_Wago:Wago_734-132_1x02_P3.50mm_Vertical" (layer "F.Cu")
+    (at 99.7 104.1)
+    (descr "Molex 734 Male header (for PCBs); Straight solder pin 1 x 1 mm, 734-132 , 2 Pins (http://www.farnell.com/datasheets/2157639.pdf), generated with kicad-footprint-generator")
+    (tags "connector Wago  side entry")
+    (property "Sheetfile" "H-brygga V3.kicad_sch")
+    (property "Sheetname" "")
+    (attr through_hole)
+    (fp_text reference "J8" (at 1.9 -5.35) (layer "F.SilkS")
+      (effects (font (size 1 1) (thickness 0.15)))
+    )
+    (fp_text value "Högtalare" (at 1.9 5.55) (layer "F.Fab")
+      (effects (font (size 1 1) (thickness 0.15)))
+    )
+    (fp_text user "${REFERENCE}" (at 1.9 3.65) (layer "F.Fab")
+      (effects (font (size 1 1) (thickness 0.15)))
+    )
+    (fp_line (start -3.21 -2.15) (end -3.21 -4.56) (layer "F.SilkS") (width 0.12))
+    (fp_line (start 0 2.85) (end 0 3.85) (layer "F.SilkS") (width 0.12))
+    (fp_line (start 3.5 3.85) (end 6.1 3.85) (layer "F.SilkS") (width 0.12))
+    (fp_line (start 6.71 -4.26) (end -2.91 -4.26) (layer "F.SilkS") (width 0.12))
+    (fp_line (start 2.6 2.85) (end 3.5 2.85) (layer "F.SilkS") (width 0.12))
+    (fp_line (start 2.6 3.85) (end 2.6 2.85) (layer "F.SilkS") (width 0.12))
+    (fp_line (start -3.21 -4.56) (end -0.8 -4.56) (layer "F.SilkS") (width 0.12))
+    (fp_line (start -2.3 2.85) (end 0 2.85) (layer "F.SilkS") (width 0.12))
+    (fp_line (start -2.91 -4.26) (end -2.91 4.46) (layer "F.SilkS") (width 0.12))
+    (fp_line (start 3.5 2.85) (end 3.5 3.85) (layer "F.SilkS") (width 0.12))
+    (fp_line (start 6.1 3.85) (end 6.1 -2.65) (layer "F.SilkS") (width 0.12))
+    (fp_line (start -2.3 -2.65) (end -2.3 2.85) (layer "F.SilkS") (width 0.12))
+    (fp_line (start -2.91 4.46) (end 6.71 4.46) (layer "F.SilkS") (width 0.12))
+    (fp_line (start 0 3.85) (end 2.6 3.85) (layer "F.SilkS") (width 0.12))
+    (fp_line (start 6.1 -2.65) (end -2.3 -2.65) (layer "F.SilkS") (width 0.12))
+    (fp_line (start 6.71 4.46) (end 6.71 -4.26) (layer "F.SilkS") (width 0.12))
+    (fp_line (start -3.3 -4.65) (end -3.3 4.85) (layer "F.CrtYd") (width 0.05))
+    (fp_line (start 7.1 4.85) (end 7.1 -4.65) (layer "F.CrtYd") (width 0.05))
+    (fp_line (start 7.1 -4.65) (end -3.3 -4.65) (layer "F.CrtYd") (width 0.05))
+    (fp_line (start -3.3 4.85) (end 7.1 4.85) (layer "F.CrtYd") (width 0.05))
+    (fp_line (start 0 -3.442893) (end 0.5 -4.15) (layer "F.Fab") (width 0.1))
+    (fp_line (start -2.8 4.35) (end 6.6 4.35) (layer "F.Fab") (width 0.1))
+    (fp_line (start -2.8 -4.15) (end -2.8 4.35) (layer "F.Fab") (width 0.1))
+    (fp_line (start -0.5 -4.15) (end 0 -3.442893) (layer "F.Fab") (width 0.1))
+    (fp_line (start 6.6 4.35) (end 6.6 -4.15) (layer "F.Fab") (width 0.1))
+    (fp_line (start 6.6 -4.15) (end -2.8 -4.15) (layer "F.Fab") (width 0.1))
+    (pad "1" thru_hole roundrect (at 0 0) (size 2 2.6) (drill 1.6) (layers *.Cu *.Mask) (roundrect_rratio 0.125)
+      (net 66 "Net-(J8-Pad1)") (pinfunction "Pin_1") (pintype "passive"))
+    (pad "2" thru_hole oval (at 3.5 0) (size 2 2.6) (drill 1.6) (layers *.Cu *.Mask)
+      (net 67 "Net-(J8-Pad2)") (pinfunction "Pin_2") (pintype "passive"))
+    (model "${KICAD6_3DMODEL_DIR}/Connector_Wago.3dshapes/Wago_734-132_1x02_P3.50mm_Vertical.wrl"
+      (offset (xyz 0 0 0))
+      (scale (xyz 1 1 1))

Commit message: H-brygga inför fräsning
Parts:
- added Q1: Q_NMOS_DGS, Package_TO_SOT_THT:TO-92_HandSolder, F.Cu at (77.6, 88.4)
- added Q2: Q_NMOS_DGS, Package_TO_SOT_THT:TO-92_HandSolder, F.Cu at (77.2, 82.7)
- U2: footprint footprints:DIPS1778W50P254L2100H170Q16N -> Egna:DIPS1778W50P254L2100H170Q16N
- moved J1 56.5 mm to (31.6, 87.2)
- moved J7 22.7 mm to (68.7, 92.8)
- moved U2 21.4 mm to (101.6, 100.5), turned to 180 degrees
- moved REF** 21.1 mm to (96.0, 118.0)
- moved R1 19.8 mm to (43.0, 96.2)
- moved R3 19.7 mm to (53.1, 99.2)
- moved D1 19.0 mm to (73.8, 88.9), turned to -90 degrees
- moved REF** 18.7 mm to (30.8, 99.3)
- moved D2 16.8 mm to (79.5, 94.0), turned to -90 degrees
- moved P2 15.3 mm to (21.6, 111.5)
- moved P1 15.1 mm to (21.6, 126.7)
- moved D3 10.4 mm to (70.5, 86.2)
- moved D4 10.3 mm to (60.5, 82.9)
- moved J5 9.98 mm to (52.4, 87.5)
- moved J8 6.55 mm to (93.8, 107.0)
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Connections:
- C3 pad 2: Net-(C3-Pad2) -> MP3+
- C4 pad 1: 7. -> 12(MISO).
- C4 pad 2: Net-(C4-Pad2) -> MP3+
- D5 pad 2: 8a -> 7a
- D6 pad 2: 8. -> 7.
- J2 pad 2: +5V -> MP3+
- J3 pad 2: +5V -> MP3+
- J4 pad 2: +5V -> MP3+
- J5 pad 2: +5V -> MP3+
- J6 pad 2: +5V -> MP3+
- P1 pad 11: 8. -> /8.
- P1 pad 15: /12(MISO). -> 12(MISO).
- P1 pad 6: /3(**). -> 3(**).
- P1 pad 8: /5(**). -> 5(**).
- P2 pad 4: +5V -> MP3+
- P7 pad 10: /7a -> 7a
- P8 pad 4: +5V -> MP3+
- R4 pad 2: 7. -> 12(MISO).
- SW1 pad 1: +5V -> MP3+
- SW1 pad 2: Net-(C3-Pad2) -> MP3+
- SW1 pad 4: unconnected-(SW1-Pad4) -> 12(MISO)
- SW2 pad 1: +5V -> MP3+
- SW2 pad 2: Net-(C4-Pad2) -> MP3+
- SW2 pad 3: 7. -> 12(MISO).
- SW2 pad 4: unconnected-(SW2-Pad4) -> 12(MISO).
- U1 pad 9: +5V -> MP3+
- U2 pad 11: Next -> Net-(U2-Pad11)
- U2 pad 9: Previous -> Net-(U2-Pad9)
Routing:
- net MP3+: track 0.00 -> 223.9 mm, vias 0 -> 4
- net +5V: track 132.6 -> 0.00 mm
- net 3(**).: track 0.00 -> 78.0 mm, vias 0 -> 2
- net GND: track 227.2 -> 299.1 mm, vias 0 -> 1
- net 5(**).: track 0.00 -> 66.5 mm, vias 0 -> 2
- net Vin: track 188.0 -> 146.4 mm
- net A0.: track 16.0 -> 56.3 mm
- net 6(**).: track 44.0 -> 5.47 mm
- net A1.: track 20.4 -> 49.1 mm
- net Net-(J8-Pad1): track 0.00 -> 27.5 mm
- net 7.: track 47.9 -> 20.9 mm
- net 7a: track 0.00 -> 21.2 mm
- net Net-(J8-Pad2): track 0.00 -> 21.0 mm
- net 8.: track 18.2 -> 0.00 mm
- net Net-(D5-Pad1): track 3.76 -> 20.9 mm
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Other:
- board size 78.2 x 63.2 mm -> 86.1 x 60 mm
