File: H-Brygga v3/H-brygga V3/H-brygga V3.kicad_pcb (KiCad board)
At the start: 2 copper layers, 86.1 x 60 mm, 35 parts, among them J1 POWER, J2 sensor vänster, J3 SERVO, J4 sensor motor, J5 START, J6 sensor höger, J7 MOTOR, J8 Högtalare, P1 Digital, P2 Analog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

Commit message: Kod bil jacob
Parts:
- J2: value sensor vänster -> sensor höger
- J6: value sensor höger -> sensor vänster
Connections:
- net MP3+ renamed +5V
Changed lines of the file:
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@@
   (net 69 "/8.")
   (net 70 "/10(**{slash}SS).")
-  (net 71 "MP3+")
+  (net 71 "+5V")
   (net 72 "5(**).")
-  (net 73 "Net-(U2-Pad11)")
-  (net 74 "Net-(U2-Pad9)")
+  (net 73 "Net-(Q1-Pad3)")
+  (net 74 "Net-(Q2-Pad3)")
   (footprint "Connector_JST:JST_XH_B3B-XH-A_1x03_P2.50mm_Vertical" (layer "F.Cu")
     (at 52.425 87.5 90)
@@
       (net 11 "5(**)") (pinfunction "Pin_1") (pintype "passive"))
     (pad "2" thru_hole oval (at 2.5 0 90) (size 1.7 1.95) (drill 0.95) (layers *.Cu *.Mask)
-      (net 71 "MP3+") (pinfunction "Pin_2") (pintype "passive"))
+      (net 71 "+5V") (pinfunction "Pin_2") (pintype "passive"))
     (pad "3" thru_hole oval (at 5 0 90) (size 1.7 1.95) (drill 0.95) (layers *.Cu *.Mask)
       (net 2 "GND") (pinfunction "Pin_3") (pintype "passive"))
@@
       (effects (font (size 1 1) (thickness 0.15)))
     )
-    (fp_text value "sensor höger" (at 2.5 4.6 90) (layer "F.Fab")
+    (fp_text value "sensor vänster" (at 2.5 4.6 90) (layer "F.Fab")
       (effects (font (size 1 1) (thickness 0.15)))
     )
@@
       (net 47 "A1.") (pinfunction "Pin_1") (pintype "passive"))
     (pad "2" thru_hole oval (at 0 0 90) (size 1.7 1.95) (drill 0.95) (layers *.Cu *.Mask)
-      (net 71 "MP3+") (pinfunction "Pin_2") (pintype "passive"))
+      (net 71 "+5V") (pinfunction "Pin_2") (pintype "passive"))
     (pad "3" thru_hole oval (at 2.5 0 90) (size 1.7 1.95) (drill 0.95) (layers *.Cu *.Mask)
       (net 2 "GND") (pinfunction "Pin_3") (pintype "passive"))
@@
       (net 2 "GND") (pinfunction "GND") (pintype "power_in"))
     (pad "9" thru_hole oval (at 10.16 0 270) (size 1.8 1.8) (drill 1) (layers *.Cu *.Mask)
-      (net 71 "MP3+") (pinfunction "Vss") (pintype "power_in"))
+      (net 71 "+5V") (pinfunction "Vss") (pintype "power_in"))
     (pad "10" thru_hole oval (at 11.43 -5.08 270) (size 1.8 1.8) (drill 1) (layers *.Cu *.Mask)
       (net 41 "unconnected-(U1-Pad10)") (pinfunction "IN3") (pintype "input"))
@@
       (net 30 "/Reset") (pinfunction "Pin_3") (pintype "passive"))
     (pad "4" thru_hole oval (at 7.62 0) (size 1.7272 2.032) (drill 1.016) (layers *.Cu *.Mask "F.SilkS")
-      (net 71 "MP3+") (pinfunction "Pin_4") (pintype "passive"))
+      (net 71 "+5V") (pinfunction "Pin_4") (pintype "passive"))
     (pad "5" thru_hole oval (at 10.16 0) (size 1.7272 2.032) (drill 1.016) (layers *.Cu *.Mask "F.SilkS")
       (net 34 "/A7") (pinfunction "Pin_5") (pintype "passive"))
@@
       (effects (font (size 1 1) (thickness 0.15)))
     )
-    (fp_text value "sensor vänster" (at 2.5 4.6 90) (layer "F.Fab")
+    (fp_text value "sensor höger" (at 2.5 4.6 90) (layer "F.Fab")
       (effects (font (size 1 1) (thickness 0.15)))
     )
@@
       (net 46 "A0.") (pinfunction "Pin_1") (pintype "passive"))
     (pad "2" thru_hole oval (at 0 0 90) (size 1.7 1.95) (drill 0.95) (layers *.Cu *.Mask)
-      (net 71 "MP3+") (pinfunction "Pin_2") (pintype "passive"))
+      (net 71 "+5V") (pinfunction "Pin_2") (pintype "passive"))
     (pad "3" thru_hole oval (at 2.5 0 90) (size 1.7 1.95) (drill 0.95) (layers *.Cu *.Mask)
       (net 2 "GND") (pinfunction "Pin_3") (pintype "passive"))
@@
       (net 72 "5(**).") (pinfunction "G") (pintype "input"))
     (pad "3" thru_hole roundrect (at 2.54 0) (size 1.1 1.8) (drill 0.75 (offset 0 0.4)) (layers *.Cu *.Mask) (roundrect_rratio 0.25)
-      (net 73 "Net-(U2-Pad11)") (pinfunction "S") (pintype "passive"))
+      (net 73 "Net-(Q1-Pad3)") (pinfunction "S") (pintype "passive"))
     (model "${KICAD6_3DMODEL_DIR}/Package_TO_SOT_THT.3dshapes/TO-92.wrl"
       (offset (xyz 0 0 0))
@@
       (net 14 "/Reset.") (pinfunction "Pin_3") (pintype "passive"))
     (pad "4" thru_hole oval (at 7.62 0) (size 1.7272 2.032) (drill 1.016) (layers *.Cu *.Mask "F.SilkS")
-      (net 71 "MP3+") (pinfunction "Pin_4") (pintype "passive"))
+      (net 71 "+5V") (pinfunction "Pin_4") (pintype "passive"))
     (pad "5" thru_hole oval (at 10.16 0) (size 1.7272 2.032) (drill 1.016) (layers *.Cu *.Mask "F.SilkS")
       (net 19 "/A7.") (pinfunction "Pin_5") (pintype "passive"))
@@
     (fp_line (start -1.61 19.39) (end -1.61 -1.61) (layer "F.Fab") (width 0.1))
     (pad "1" thru_hole rect (at 0 0 180) (size 1.35 1.35) (drill 0.9) (layers *.Cu *.Mask)
-      (net 71 "MP3+") (pinfunction "VCC") (pintype "power_in"))
+      (net 71 "+5V") (pinfunction "VCC") (pintype "power_in"))
     (pad "2" thru_hole circle (at 0 2.54 180) (size 1.35 1.35) (drill 0.9) (layers *.Cu *.Mask)
       (net 54 "unconnected-(U2-Pad2)") (pinfunction "RX") (pintype "input"))
@@
       (net 52 "Net-(J8-Pad1)") (pinfunction "SPK_2") (pintype "output"))
     (pad "9" thru_hole circle (at 17.78 17.78 180) (size 1.35 1.35) (drill 0.9) (layers *.Cu *.Mask)
-      (net 74 "Net-(U2-Pad9)") (pinfunction "IO_1") (pintype "input"))
+      (net 74 "Net-(Q2-Pad3)") (pinfunction "IO_1") (pintype "input"))
     (pad "10" thru_hole circle (at 17.78 15.24 180) (size 1.35 1.35) (drill 0.9) (layers *.Cu *.Mask)
       (net 2 "GND") (pinfunction "GND_2") (pintype "power_in"))
     (pad "11" thru_hole circle (at 17.78 12.7 180) (size 1.35 1.35) (drill 0.9) (layers *.Cu *.Mask)
-      (net 73 "Net-(U2-Pad11)") (pinfunction "IO_2") (pintype "input"))
+      (net 73 "Net-(Q1-Pad3)") (pinfunction "IO_2") (pintype "input"))
     (pad "12" thru_hole circle (at 17.78 10.16 180) (size 1.35 1.35) (drill 0.9) (layers *.Cu *.Mask)
       (net 58 "unconnected-(U2-Pad12)") (pinfunction "ADKEY_1") (pintype "input"))
@@
     (fp_line (start 6.25 -0.75) (end 6.25 5.25) (layer "F.Fab") (width 0.1))
     (pad "1" thru_hole rect (at 0 0 270) (size 1.7 1.7) (drill 1) (layers *.Cu *.Mask)
-      (net 71 "MP3+") (pinfunction "1") (pintype "passive"))
+      (net 71 "+5V") (pinfunction "1") (pintype "passive"))
     (pad "2" thru_hole circle (at 6.5 0 270) (size 1.7 1.7) (drill 1) (layers *.Cu *.Mask)
-      (net 71 "MP3+") (pinfunction "2") (pintype "passive"))
+      (net 71 "+5V") (pinfunction "2") (pintype "passive"))
     (pad "3" thru_hole circle (at 0 4.5 270) (size 1.7 1.7) (drill 1) (layers *.Cu *.Mask)
       (net 50 "12(MISO)") (pinfunction "K") (pintype "passive"))
@@
       (net 65 "3(**).") (pinfunction "G") (pintype "input"))
     (pad "3" thru_hole roundrect (at 2.54 0) (size 1.1 1.8) (drill 0.75 (offset 0 0.4)) (layers *.Cu *.Mask) (roundrect_rratio 0.25)
-      (net 74 "Net-(U2-Pad9)") (pinfunction "S") (pintype "passive"))
+      (net 74 "Net-(Q2-Pad3)") (pinfunction "S") (pintype "passive"))
     (model "${KICAD6_3DMODEL_DIR}/Package_TO_SOT_THT.3dshapes/TO-92.wrl"
       (offset (xyz 0 0 0))
@@
       (net 10 "A1") (pinfunction "Pin_1") (pintype "passive"))
     (pad "2" thru_hole oval (at 2.5 0 90) (size 1.7 1.95) (drill 0.95) (layers *.Cu *.Mask)
-      (net 71 "MP3+") (pinfunction "Pin_2") (pintype "passive"))
+      (net 71 "+5V") (pinfunction "Pin_2") (pintype "passive"))
     (pad "3" thru_hole oval (at 5 0 90) (size 1.7 1.95) (drill 0.95) (layers *.Cu *.Mask)
       (net 2 "GND") (pinfunction "Pin_3") (pintype "passive"))
@@
       (net 50 "12(MISO)") (pintype "passive"))
     (pad "2" thru_hole circle (at 2.5 0 270) (size 1.4 1.4) (drill 0.7) (layers *.Cu *.Mask)
-      (net 71 "MP3+") (pintype "passive"))
+      (net 71 "+5V") (pintype "passive"))
     (model "${KICAD6_3DMODEL_DIR}/Capacitor_THT.3dshapes/C_Rect_L4.6mm_W2.0mm_P2.50mm_MKS02_FKP02.wrl"
       (offset (xyz 0 0 0))
@@
     (fp_line (start 0.25 -0.75) (end 0.25 5.25) (layer "F.Fab") (width 0.1))
     (pad "1" thru_hole rect (at 0 0 180) (size 1.7 1.7) (drill 1) (layers *.Cu *.Mask)
-      (net 71 "MP3+") (pinfunction "1") (pintype "passive"))
+      (net 71 "+5V") (pinfunction "1") (pintype "passive"))
     (pad "2" thru_hole circle (at 6.5 0 180) (size 1.7 1.7) (drill 1) (layers *.Cu *.Mask)
-      (net 71 "MP3+") (pinfunction "2") (pintype "passive"))
+      (net 71 "+5V") (pinfunction "2") (pintype "passive"))
     (pad "3" thru_hole circle (at 0 4.5 180) (size 1.7 1.7) (drill 1) (layers *.Cu *.Mask)
       (net 68 "12(MISO).") (pinfunction "K") (pintype "passive"))
@@
       (net 68 "12(MISO).") (pintype "passive"))
     (pad "2" thru_hole circle (at 2.5 0 270) (size 1.4 1.4) (drill 0.7) (layers *.Cu *.Mask)
-      (net 71 "MP3+") (pintype "passive"))
+      (net 71 "+5V") (pintype "passive"))
     (model "${KICAD6_3DMODEL_DIR}/Capacitor_THT.3dshapes/C_Rect_L4.6mm_W2.0mm_P2.50mm_MKS02_FKP02.wrl"
       (offset (xyz 0 0 0))
@@
       (net 9 "6(**).") (pinfunction "Pin_1") (pintype "passive"))
     (pad "2" thru_hole oval (at 0 0 90) (size 1.7 1.95) (drill 0.95) (layers *.Cu *.Mask)
-      (net 71 "MP3+") (pinfunction "Pin_2") (pintype "passive"))
+      (net 71 "+5V") (pinfunction "Pin_2") (pintype "passive"))
     (pad "3" thru_hole oval (at 2.5 0 90) (size 1.7 1.95) (drill 0.95) (layers *.Cu *.Mask)
       (net 2 "GND") (pinfunction "Pin_3") (pintype "passive"))
