File: H-Brygga v3/H-brygga V3/H-brygga V3.kicad_sch (KiCad schematic)
At the start: 39 parts, among them J1 POWER, J2 sensor vänster, J3 SERVO, J4 sensor motor, J5 START, J6 sensor höger, J7 MOTOR, P1 Digital, P10 CONN_01X01, P11 CONN_01X01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

Commit message: H-brygga inför fräsning
Parts:
- removed P10, P11, P12, P3, P4, P5, P6, P9: CONN_01X01, Socket_Arduino_Nano:1pin_Nano, symbol Connector_Generic:Conn_01x01
- added Q1: (no value), symbol Device:Q_NMOS_DGS
- added Q2: Q_NMOS_DGS, Package_TO_SOT_THT:TO-92_HandSolder, symbol Device:Q_NMOS_DGS
- J8: value (none) -> Högtalare
Connections:
- net MP3+ is gone; now on net +5V: U2.1 (VCC)
- net +5V: now also C3.2, C4.2, SW1.2, SW2.2
- net 12(MISO): now also SW1.4 (A)
- net 12(MISO).: now also C4.1, R4.2, SW2.3 (K), SW2.4 (A)
- net 3(**).: now also Q2.2 (G)
- net 5(**).: now also Q1.2 (G)
- net 7.: now also D6.2 (A); no longer C4.1, R4.2, SW2.3 (K)
- net 7a: now also D5.2 (A)
- net 8.: no longer D6.2 (A)
- net 8a: no longer D5.2 (A)
- net GND: now also Q1.1 (D), Q2.1 (D)
- net Next: no longer names the net of U2.11 (IO_2)
- net Next: now also Q1.3 (S)
- net Previous: no longer names the net of U2.9 (IO_1)
- net Previous: now also Q2.3 (S)
- no-connect marks 8 -> 0
Other:
- moved on the sheet: C3, C4, J8, R2, R4, SW1, SW2, U2

Commit message: Kod bil jacob
Parts:
- J2: value sensor vänster -> (none)
- J6: value sensor höger -> (none)
- Q1: value (none) -> Q_NMOS_DGS; footprint (none) -> Package_TO_SOT_THT:TO-92_HandSolder
- U2: value (none) -> DFR0299; footprint (none) -> Egna:DIPS1778W50P254L2100H170Q16N
Changed lines of the file:
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@@
       (effects (font (size 1.27 1.27)) (justify left))
     )
-    (property "Value" "" (id 1) (at 174.625 33.6549 0)
-      (effects (font (size 1.27 1.27)) (justify left))
-    )
-    (property "Footprint" "" (id 2) (at 173.355 29.845 0)
+    (property "Value" "Q_NMOS_DGS" (id 1) (at 174.625 33.6549 0)
+      (effects (font (size 1.27 1.27)) (justify left))
+    )
+    (property "Footprint" "Package_TO_SOT_THT:TO-92_HandSolder" (id 2) (at 173.355 29.845 0)
       (effects (font (size 1.27 1.27)) hide)
     )
@@
       (effects (font (size 1.27 1.27)) (justify left))
     )
-    (property "Value" "sensor vänster" (id 1) (at 26.416 83.566 90)
+    (property "Value" "" (id 1) (at 26.416 83.566 90)
       (effects (font (size 1.27 1.27)) (justify left))
     )
@@
     (in_bom yes) (on_board yes)
     (property "Reference" "U2" (id 0) (at 131.445 20.193 0))
-    (property "Value" "" (id 1) (at 131.445 22.733 0))
-    (property "Footprint" "" (id 2) (at 144.145 24.765 0)
+    (property "Value" "DFR0299" (id 1) (at 131.445 22.733 0))
+    (property "Footprint" "Egna:DIPS1778W50P254L2100H170Q16N" (id 2) (at 144.145 24.765 0)
       (effects (font (size 1.27 1.27)) (justify left) hide)
     )
@@
       (effects (font (size 1.27 1.27)) (justify left))
     )
-    (property "Value" "sensor höger" (id 1) (at 53.086 83.82 90)
+    (property "Value" "" (id 1) (at 53.086 83.82 90)
       (effects (font (size 1.27 1.27)) (justify left))
     )
@@
     )
     (path "/557efbe0-59d9-4c3b-875e-681f1d0eabac"
-      (reference "J2") (unit 1) (value "sensor vänster") (footprint "Connector_JST:JST_XH_B3B-XH-A_1x03_P2.50mm_Vertical")
+      (reference "J2") (unit 1) (value "sensor höger") (footprint "Connector_JST:JST_XH_B3B-XH-A_1x03_P2.50mm_Vertical")
     )
     (path "/3de27c1c-897a-4a6c-b0f7-6b3c6fd91fd1"
@@
     )
     (path "/d0583253-7f1c-498c-afba-93bf9b28c781"
-      (reference "J6") (unit 1) (value "sensor höger") (footprint "Connector_JST:JST_XH_B3B-XH-A_1x03_P2.50mm_Vertical")
+      (reference "J6") (unit 1) (value "sensor vänster") (footprint "Connector_JST:JST_XH_B3B-XH-A_1x03_P2.50mm_Vertical")
     )
     (path "/a5c7f988-1d57-48d4-82d1-1deaeac9e184"
